File: kicad/WakeCircuit/WakeCircuit.kicad_pcb (KiCad board)
At the start: 2 copper layers, 34 x 21.2 mm, 16 parts, among them J1 Conn_01x12_Socket, J2 Conn_01x10_Socket, J4 Conn_01x03_Socket, U1 TLV7011DBVR, U3 4013

Commit message: Update missing component 3d cad files
Parts:
- moved RV1 14.8 mm to (95.3, 111.9)
- moved R1 7.20 mm to (101.8, 102.2)
- moved U1 5.56 mm to (108.0, 103.0)
- moved J4 2.01 mm to (98.2, 102.8)
Routing:
- net Net-(U1-IN-): track 2.34 -> 28.2 mm, vias 0 -> 2
- net +3V3: track 76.3 -> 68.0 mm
- net Net-(U1-OUT): track 30.5 -> 25.1 mm
- net LDR_SIG: track 8.90 -> 10.3 mm
- net GND: track 16.0 -> 14.8 mm
- net GPIO_1: track 44.4 -> 45.4 mm
Other:
- board text added: "1"
